File: PCB/EC60_PCB/matrix.kicad_sch (KiCad schematic)
At the start: 74 parts, among them SW10 EC_SW, SW11 EC_SW, SW12 EC_SW, SW13 EC_SW, SW14 EC_SW, SW15 EC_SW, SW16 EC_SW, SW17 EC_SW, SW18 EC_SW, SW19 EC_SW, SW2 EC_SW, SW20 EC_SW, SW21 EC_SW, SW22 EC_SW, SW23 EC_SW, SW24 EC_SW, SW25 EC_SW, SW26 EC_SW, SW27 EC_SW, SW28 EC_SW, SW29 EC_SW, SW3 EC_SW, SW30 EC_SW, SW31 ANSI_\, SW32 ISO_Enter, SW33 EC_SW, SW34 EC_SW, SW35 EC_SW, SW36 EC_SW, SW37 EC_SW, SW38 EC_SW, SW39 EC_SW, SW4 EC_SW, SW40 EC_SW, SW41 EC_SW, SW42 EC_SW, SW43 EC_SW, SW44 EC_SW, SW45 ISO_|, SW46 ANSI_Enter, SW47 EC_SW, SW48 EC_SW, SW49 EC_SW, SW5 EC_SW, SW50 EC_SW, SW51 EC_SW, SW52 EC_SW, SW53 EC_SW, SW54 EC_SW, SW55 EC_SW, SW56 EC_SW, SW57 EC_SW, SW58 EC_SW, SW59 EC_SW, SW6 EC_SW, SW60 EC_SW_1u&1.75u, SW61 EC_SW, SW62 EC_SW_1u&1.75u, SW63 EC_SW, SW64 EC_SW, SW65 EC_SW, SW66 EC_SW, SW67 EC_SW, SW68 EC_SW, SW69 EC_SW, SW7 EC_SW, SW70 EC_SW, SW71 EC_SW, SW72 EC_SW, SW73 EC_SW, SW74 EC_SW, SW75 EC_SW, SW8 EC_SW, SW9 EC_SW

Commit message: Update for 3d models
Parts:
- SW10, SW11, SW12, SW13, SW14, SW15, SW17, SW18, SW19, SW2, SW20, SW21, SW22, SW23, SW24, SW25, SW26, SW27, SW28, SW29, SW3, SW30, SW31, SW34, SW35, SW36, SW37, SW38, SW39, SW4, SW40, SW41, SW42, SW43, SW44, SW45, SW47, SW5, SW50, SW51, SW52, SW53, SW54, SW55, SW56, SW57, SW58, SW59, SW6, SW63, SW64, SW65, SW66, SW67, SW7, SW70, SW72, SW73, SW74, SW75, SW8, SW9: footprint cipulot_parts:ecs_pad_no_ring -> cipulot_parts:ecs_pad_1U_no_ring
- SW16, SW32, SW46, SW61: footprint cipulot_parts:ecs_pad_no_ring -> cipulot_parts:ecs_pad_2U_no_ring
- SW48, SW49: footprint cipulot_parts:ecs_pad_no_ring_1u_edge_cut -> cipulot_parts:ecs_pad_1U_no_ring_1u_edge_cut
